File: mixpower-profiler-hv-module-v2.kicad_sch (KiCad schematic)
At the start: 70 parts, among them J1 VIN_TERMINAL, J2 VIN_HEADERS, J3 COMM_HEADERS, Q1 STL130N6F7, Q2 STL130N6F7, Q3 STL130N6F7, Q4 STL130N6F7, Q5 STL130N6F7, Q6 STL130N6F7, U1 FAN73711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

Commit message: feat: add PTC fuse on VIN
Parts:
- added F1: Polyfuse_Small, Resistor_SMD:R_1812_4532Metric, symbol Device:Polyfuse_Small
Connections:
- net VIN_P: now also F1.2; no longer D7.1 (A1), J1.1 (Pin_1), J2.1 (Pin_1), J2.2 (Pin_2)
- new net VIN_P_IN: D7.1 (A1), F1.1, J1.1 (Pin_1), J2.1 (Pin_1), J2.2 (Pin_2)
Other:
- moved on the sheet: C1, C2, C3, C4, C5, C6, C7, C8, C9, D1, D2, D3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
